File: dcpsu-card-b.kicad_pcb (KiCad board)
At the start: 2 copper layers, 80 x 105 mm, 91 parts, among them J1 PCIe_x1, J2 AVR-ISP-6, J3 Conn_01x06, J4 Conn_01x01_Female, J5 Conn_01x01_Female, Q1 SSM6N7002KFU,LF, U1 ATtiny87-MU, U10 INA219AIDCNR, U2 NCP5623, U3 LM358DR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

Commit message: Update with notes and pending changes
Other:
- board text added: "FIX edge conn footprint"
- board text added: "FIX feedback layout"
- board text added: "FIX feedback net"
Changed lines of the file:
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@@
   (general
     (thickness 1.6)
-    (drawings 46)
+    (drawings 49)
     (tracks 657)
     (zones 0)
@@
       (xy -1.971615 -1.454739) (xy -1.908759 -1.469184)) (layer B.SilkS) (width 0.01))
   )
+  (gr_text "FIX feedback net" (at 92 92) (layer Cmts.User)
+    (effects (font (size 1.5 1.5) (thickness 0.3)))
+  )
+  (gr_text "FIX feedback layout" (at 84 102) (layer Cmts.User)
+    (effects (font (size 1.5 1.5) (thickness 0.3)))
+  )
+  (gr_text "FIX edge conn footprint" (at 62 93) (layer Cmts.User)
+    (effects (font (size 1.5 1.5) (thickness 0.3)))
+  )
   (gr_text "Open Source Hardware\n© Kyle E\nLicense: CreativeCommons BY-SA" (at 100 130) (layer B.Cu)
