File: dcpsu-card-b.sch (KiCad schematic (older format))
At the start: 70 parts, among them Q1 SSM6N7002KFU,LF, U1 ATtiny87-MU, U10 INA219AIDCNR, U3 LM358DR, U4 MCP47FEB22A0T-E_ST, U5 AOZ2151PQI-10, U6 LM358DR, U7 MCP4017T-104E_LT, U8 LD1084, U9 LM334M

Commit message: Card A Rev 0.3
Parts:
- removed R9: 2k, Resistor_SMD:R_0603_1608Metric_Pad1.05x0.95mm_HandSolder, symbol Device:R
- C11, C8: Digi-Key_PN 399-1099-1-ND -> 1276-1000-1-ND
- C7: value 1u -> 10u; Digi-Key_PN 399-7847-1-ND -> 478-10766-1-ND
Changed lines of the file:
@@
 PWR-EN
-$Comp
-L power:+5V #PWR026
-U 1 1 5EB29CED
-P 5100 700
-F 0 "#PWR026" H 5100 550 50  0001 C CNN
-F 1 "+5V" H 5115 873 50  0000 C CNN
-F 2 "" H 5100 700 50  0001 C CNN
-F 3 "" H 5100 700 50  0001 C CNN
-	1    5100 700
-	1    0    0    -1
-$EndComp
 $Comp
 L Device:C C7
@@
 P 4900 1150
 F 0 "C7" H 5015 1196 50  0000 L CNN
-F 1 "1u" H 5015 1105 50  0000 L CNN
+F 1 "10u" H 5015 1105 50  0000 L CNN
 F 2 "Capacitor_SMD:C_0603_1608Metric_Pad1.05x0.95mm_HandSolder" H 4938 1000 50  0001 C CNN
 F 3 "" H 4900 1150 50  0001 C CNN
-F 4 "399-7847-1-ND" H 0   0   50  0001 C CNN "Digi-Key_PN"
+F 4 "478-10766-1-ND" H 0   0   50  0001 C CNN "Digi-Key_PN"
 	1    4900 1150
 	0    -1   -1   0
@@
 F 2 "Capacitor_SMD:C_0603_1608Metric_Pad1.05x0.95mm_HandSolder" H 6538 1200 50  0001 C CNN
 F 3 "" H 6500 1350 50  0001 C CNN
-F 4 "399-1099-1-ND" H 0   0   50  0001 C CNN "Digi-Key_PN"
+F 4 "1276-1000-1-ND" H 0   0   50  0001 C CNN "Digi-Key_PN"
 	1    6500 1350
 	1    0    0    -1
@@
 F 2 "Capacitor_SMD:C_0603_1608Metric_Pad1.05x0.95mm_HandSolder" H 5088 1900 50  0001 C CNN
 F 3 "" H 5050 2050 50  0001 C CNN
-F 4 "399-1099-1-ND" H 5050 2050 50  0001 C CNN "Digi-Key_PN"
+F 4 "1276-1000-1-ND" H 5050 2050 50  0001 C CNN "Digi-Key_PN"
 	1    5050 2050
 	1    0    0    -1
@@
 Wire Wire Line
 	2250 1600 2250 1200
-$Comp
-L Device:R R9
-U 1 1 5F7DE9F0
-P 5100 900
-F 0 "R9" H 5170 946 50  0000 L CNN
-F 1 "2k" H 5170 855 50  0000 L CNN
-F 2 "Resistor_SMD:R_0603_1608Metric_Pad1.05x0.95mm_HandSolder" V 5030 900 50  0001 C CNN
-F 3 "~" H 5100 900 50  0001 C CNN
-F 4 "RMCF0603FT2K00CT-ND" H 0   0   50  0001 C CNN "Digi-Key_PN"
-	1    5100 900
-	1    0    0    -1
-$EndComp
-Wire Wire Line
-	5050 1150 5100 1150
-Wire Wire Line
-	5100 1150 5100 1050
-Connection ~ 5100 1150
 Wire Wire Line
 	4750 1150 4700 1150
 Wire Wire Line
 	4700 1150 4700 1200
-Wire Wire Line
-	5100 750  5100 700
-Wire Wire Line
-	5100 1150 5250 1150
 Wire Wire Line
 	10200 3700 10400 3700
@@
 	-1   0    0    1
 $EndComp
+Wire Wire Line
+	5050 1150 5250 1150
 $EndSCHEMATC

Commit message: Update with notes and pending changes
Other:
- note added: "2.048V"
- note added: "64mV/R=Iset\nIset >= 3mA\nR <= 21ohm"
- note added: "FIX: VREF decoupling cap"
- note added: "FIX: alternative buck controllers with better footprint"
- note added: "FIX: card edge footprint is wrong"
- note added: "FIX: output caps"
- note added: "FIX: replace with dac"
- note added: "FIX: ~SHDN~ pin should be high"
- note added: "LD1084 uses feedback relative to fixed ref voltage"
- note added: "MCP47FEB uses same addr range as MCP4706"
- note added: "TEST POINTS!"
- note added: "V Amp\nGain = 10\n0 to 20.48V"
- note added: "comparator"
- note added: "replace with diff amp IC?"
Changed lines of the file:
@@
 Wire Wire Line
 	5050 1150 5250 1150
+Text Notes 6450 3100 0    50   ~ 0
+FIX: replace with dac
+Text Notes 3900 5450 0    50   ~ 0
+MCP47FEB uses same addr range as MCP4706
+Text Notes 4150 3350 0    50   ~ 0
+TEST POINTS!
+Text Notes 4200 2550 0    50   ~ 0
+FIX: alternative buck controllers with better footprint
+Text Notes 2550 1550 0    50   ~ 0
+FIX: card edge footprint is wrong
+Text Notes 3750 4850 0    50   ~ 0
+FIX: VREF decoupling cap
+Text Notes 5550 5250 0    50   ~ 0
+FIX: output caps
+Text Notes 2250 3150 0    50   ~ 0
+FIX: ~SHDN~ pin should be high
+Text Notes 9950 6050 0    50   ~ 0
+64mV/R=Iset\nIset >= 3mA\nR <= 21ohm
+Text Notes 4200 7050 0    50   ~ 0
+replace with diff amp IC?
+Text Notes 6700 5900 0    50   ~ 0
+comparator
+Text Notes 6900 4850 0    50   ~ 0
+V Amp\nGain = 10\n0 to 20.48V
+Text Notes 3700 2600 0    50   ~ 0
+2.048V
+Text Notes 8500 3600 0    50   ~ 0
+LD1084 uses feedback relative to fixed ref voltage
 $EndSCHEMATC
