File: dcpsu-card-a.kicad_pcb (KiCad board)
At the start: 2 copper layers, 80 x 100 mm, 54 parts, among them J1 PCIe_x1, J2 Conn_01x06, J3 AVR-ISP-6, J4 Conn_01x02, U1 ATtiny87-MU, U2 AOZ2151PQI-10, U3 MCP4017T-104E_LT, U4 INA219AIDCNR

Commit message: Card A Rev 0.3
Parts:
- added C16: 0.1u, Capacitor_SMD:C_0603_1608Metric_Pad1.05x0.95mm_HandSolder, F.Cu at (96.0, 65.0)
- added R23: 100, Resistor_SMD:R_0603_1608Metric_Pad1.05x0.95mm_HandSolder, F.Cu at (91.0, 102.0)
- C2: value 1u -> 10u
- J1: footprint Connector_PCBEdge:BUS_PCIexpress -> custom-footprints:BUS_PCIe_custom
- R10, R8: value 2k -> 0
- R20: value 2k -> 3k
- R6: value 2k -> 10k
- R9: value 2k -> 47k
- RN2: footprint Resistor_SMD:R_Array_Convex_4x1206 -> Resistor_SMD:R_Array_Convex_4x0612
- U3: value MCP4017T-104E_LT -> MCP4706A0T-E_CH; footprint digikey-footprints:SOT-363 -> digikey-footprints:SOT-23-6
- moved R20 68.8 mm to (98.5, 89.0)
- moved C9 34.5 mm to (96.0, 69.0)
- moved U3 33.1 mm to (99.0, 67.0), turned to 270 degrees
- moved R10 32.2 mm to (100.0, 92.5), turned to 270 degrees
- moved R9 31.5 mm to (100.0, 89.0), turned to 270 degrees
- moved C12 20.7 mm to (127.0, 100.0), turned to 90 degrees
- moved C10 20.6 mm to (127.0, 95.0), turned to 270 degrees
- moved R7 19.0 mm to (100.0, 96.5), turned to 270 degrees
- moved R8 16.8 mm to (98.5, 96.5), turned to 90 degrees
- moved C11 16.8 mm to (124.0, 100.0), turned to 90 degrees
- moved C8 16.7 mm to (124.0, 95.0), turned to 270 degrees
- moved R3 8.25 mm to (106.0, 89.0)
- moved R14 6.41 mm to (130.0, 90.0)
- moved C15 6.14 mm to (129.0, 81.0), turned to 180 degrees
- moved C14 5.76 mm to (131.0, 87.0)
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Connections:
- C10 pad 1: GND -> GNDPWR
- C11 pad 1: GND -> GNDPWR
- C12 pad 1: GND -> GNDPWR
- C13 pad 2: GND -> GNDPWR
- C2 pad 1: Net-(C2-Pad1) -> GNDA
- C2 pad 2: GND -> Net-(C2-Pad2)
- C4 pad 2: GND -> GNDA
- C6 pad 2: GND -> GNDPWR
- C7 pad 2: GND -> GNDPWR
- C8 pad 1: GND -> GNDPWR
- D1 pad 2: GND -> GNDPWR
- J1 pad A1: GND -> GNDPWR
- J1 pad A2: +24V -> Net-(J1-PadA2)
- J1 pad B1: GND -> GNDPWR
- J1 pad B10: GND -> GNDPWR
- J1 pad B11: GND -> GNDA
- J1 pad B2: GND -> GNDPWR
- J1 pad B3: GND -> GNDPWR
- J1 pad B4: GND -> GNDPWR
- J1 pad B5: GND -> GNDPWR
- J1 pad B6: GND -> GNDPWR
- J1 pad B7: GND -> GNDPWR
- J1 pad B8: GND -> GNDPWR
- J1 pad B9: GND -> GNDPWR
- J4 pad 2: GND -> GNDPWR
- R16 pad 1: GND -> GNDPWR
- R20 pad 1: /LED1 -> Net-(R20-Pad1)
- R20 pad 2: GND -> Net-(C16-Pad1)
- R6 pad 1: +5V -> Net-(R10-Pad2)
- R6 pad 2: Net-(C2-Pad1) -> Net-(R20-Pad1)
- R7 pad 1: GND -> Net-(R10-Pad2)
- R8 pad 2: Net-(R8-Pad2) -> GNDA
- R9 pad 1: Net-(D1-Pad1) -> Net-(C10-Pad2)
- U2 pad 10: GND -> GNDPWR
- U2 pad 11: GND -> GNDPWR
- U2 pad 12: GND -> GNDPWR
- U2 pad 17: Net-(C2-Pad1) -> Net-(C2-Pad2)
- U2 pad 2: Net-(R8-Pad2) -> Net-(R10-Pad2)
- U2 pad 3: GND -> GNDA
- U3 pad 1: +5V -> Net-(C16-Pad1)
- U3 pad 3: /SCL -> +5V
- U3 pad 5: Net-(R8-Pad2) -> /SCL
- U3 pad 6: Net-(R10-Pad2) -> Net-(U3-Pad6)
Routing:
- net Net-(R8-Pad2): track 35.0 -> 0.00 mm, vias 2 -> 0
- net Net-(C10-Pad2): track 0.05 -> 26.2 mm, vias 0 -> 2
- net Net-(C16-Pad1): track 0.00 -> 26.0 mm, vias 0 -> 2
- net +5V: track 67.9 -> 43.9 mm, vias 12 -> 9
- net GND: track 61.3 -> 40.8 mm, vias 57 -> 8
- net GNDA: track 0.00 -> 20.1 mm, vias 0 -> 2
- net /PWR-PWM: track 44.4 -> 34.7 mm, vias 2 -> 4
- net /SDA: track 42.4 -> 49.7 mm
- net Net-(J1-PadA2): track 0.00 -> 6.95 mm
- net Net-(C2-Pad1): track 5.57 -> 0.00 mm
- net Net-(R10-Pad2): track 2.87 -> 6.71 mm
- net Net-(C2-Pad2): track 0.00 -> 2.49 mm
- net Net-(C4-Pad1): track 4.71 -> 2.59 mm
- net Net-(C5-Pad1): track 4.09 -> 2.17 mm
- net /SCL: track 48.6 -> 50.5 mm, vias 4 -> 3
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- added copper zone on B.Cu, net GNDA
- added copper zone on B.Cu, net GNDPWR
- added copper zone on F.Cu, net GNDPWR
- removed copper zone on F.Cu, net GND
Other:
- board text added: "DCPSU Card A v0.3"
- board text removed: "DCPSU Card A v0.1"

Commit message: Card A v0.4-WIP
Parts:
- removed C12: 22u, Capacitor_SMD:C_1206_3216Metric_Pad1.42x1.75mm_HandSolder
- removed Jx1: PinHeader_1x02_P2.54mm_Vertical, Connector_PinHeader_2.54mm:PinHeader_1x02_P2.54mm_Vertical
- removed RN2: 220, Resistor_SMD:R_Array_Convex_4x0612
- added ?: R_1206_3216Metric_Pad1.42x1.75mm_HandSolder, Resistor_SMD:R_1206_3216Metric_Pad1.42x1.75mm_HandSolder, F.Cu at (93.5, 81.0)
- added ?: R_1206_3216Metric_Pad1.42x1.75mm_HandSolder, Resistor_SMD:R_1206_3216Metric_Pad1.42x1.75mm_HandSolder, F.Cu at (93.5, 78.5)
- added ?: R_1206_3216Metric_Pad1.42x1.75mm_HandSolder, Resistor_SMD:R_1206_3216Metric_Pad1.42x1.75mm_HandSolder, F.Cu at (98.5, 67.5)
- added ?: R_1206_3216Metric_Pad1.42x1.75mm_HandSolder, Resistor_SMD:R_1206_3216Metric_Pad1.42x1.75mm_HandSolder, F.Cu at (103.5, 86.5)
- added ?: R_1206_3216Metric_Pad1.42x1.75mm_HandSolder, Resistor_SMD:R_1206_3216Metric_Pad1.42x1.75mm_HandSolder, F.Cu at (106.0, 86.5)
- added R24: 2k, Resistor_SMD:R_0603_1608Metric_Pad1.05x0.95mm_HandSolder, F.Cu at (154.0, 51.0)
- added R25: 2k, Resistor_SMD:R_0603_1608Metric_Pad1.05x0.95mm_HandSolder, F.Cu at (154.0, 53.0)
- C10, C8: value 22u -> 10u
- C11: value 22u -> 100u; footprint Capacitor_SMD:C_1206_3216Metric_Pad1.42x1.75mm_HandSolder -> Capacitor_SMD:CP_Elec_6.3x7.7
- R10: value 0 -> 3k
- R16: value 18k 0.1% -> 1k 0.1%
- R9: value 47k -> 43k
- moved C9 28.8 mm to (120.0, 85.0), turned to 180 degrees
- moved C16 28.3 mm to (116.0, 85.0), turned to 0 degrees
- moved U3 24.2 mm to (118.0, 82.0), turned to 0 degrees
- moved J2 22.8 mm to (113.0, 46.0)
- moved J3 15.3 mm to (98.0, 50.0)
- moved C3 14.0 mm to (110.0, 46.0)
- moved C1 12.7 mm to (104.5, 73.5)
- moved U1 12.3 mm to (99.8, 74.8)
- moved R1 11.5 mm to (100.5, 80.0)
- moved C1 11.5 mm to (95.5, 75.0)
- moved R5 9.85 mm to (111.0, 71.0), turned to 180 degrees
- moved R4 6.32 mm to (111.0, 69.0), turned to 180 degrees
- moved C11 4.27 mm to (125.5, 104.0), turned to 270 degrees
- moved R2 3.91 mm to (106.0, 92.0), turned to 180 degrees
- moved C15 2.24 mm to (131.0, 80.0), turned to 270 degrees
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Connections:
- C10 pad 1: GNDPWR -> Net-(C10-Pad1)
- C10 pad 2: Net-(C10-Pad2) -> GND
- C11 pad 1: GNDPWR -> Net-(C10-Pad1)
- C11 pad 2: Net-(C10-Pad2) -> GND
- C13 pad 2: GNDPWR -> GND
- C2 pad 1: GNDA -> GND
- C4 pad 2: GNDA -> GND
- C6 pad 2: GNDPWR -> GND
- C7 pad 2: GNDPWR -> GND
- C8 pad 1: GNDPWR -> Net-(C10-Pad1)
- C8 pad 2: Net-(C10-Pad2) -> GND
- D1 pad 2: GNDPWR -> GND
- D2 pad 1: Net-(D2-Pad1) -> /LED2
- D2 pad 2: GND -> Net-(D2-Pad2)
- J1 pad A1: GNDPWR -> GND
- J1 pad B1: GNDPWR -> GND
- J1 pad B10: GNDPWR -> GND
- J1 pad B11: GNDA -> GND
- J1 pad B2: GNDPWR -> GND
- J1 pad B3: GNDPWR -> GND
- J1 pad B4: GNDPWR -> GND
- J1 pad B5: GNDPWR -> GND
- J1 pad B6: GNDPWR -> GND
- J1 pad B7: GNDPWR -> GND
- J1 pad B8: GNDPWR -> GND
- J1 pad B9: GNDPWR -> GND
- J4 pad 2: GNDPWR -> GND
- L1 pad 2: Net-(C10-Pad2) -> Net-(C10-Pad1)
- R11 pad 1: Net-(C10-Pad2) -> Net-(C10-Pad1)
- R12 pad 1: Net-(C10-Pad2) -> Net-(C10-Pad1)
- R13 pad 1: Net-(C10-Pad2) -> Net-(C10-Pad1)
- R14 pad 2: Net-(C10-Pad2) -> Net-(C10-Pad1)
- R16 pad 1: GNDPWR -> GND
- R6 pad 1: Net-(R10-Pad2) -> Net-(R10-Pad1)
- R7 pad 1: Net-(R10-Pad2) -> Net-(R10-Pad1)
- R8 pad 2: GNDA -> GND
- R9 pad 1: Net-(C10-Pad2) -> Net-(R10-Pad2)
- R9 pad 2: Net-(R10-Pad1) -> Net-(C10-Pad1)
- U2 pad 10: GNDPWR -> GND
- U2 pad 11: GNDPWR -> GND
- U2 pad 12: GNDPWR -> GND
- U2 pad 2: Net-(R10-Pad2) -> Net-(R10-Pad1)
- U2 pad 3: GNDA -> GND
Routing:
- net Net-(C3-Pad2): track 32.9 -> 3.36 mm
- net Net-(C10-Pad2): track 26.2 -> 0.00 mm, vias 2 -> 0
- net /~RESET: track 44.6 -> 70.7 mm, vias 2 -> 3
- net +5V: track 43.9 -> 21.0 mm, vias 9 -> 5
- net GNDA: track 20.1 -> 0.00 mm, vias 2 -> 0
- net /LED2: track 49.0 -> 68.1 mm
- net CARD-MISO: track 66.0 -> 48.2 mm, vias 2 -> 0
- net Net-(C10-Pad1): track 0.00 -> 16.5 mm
- net /SCL: track 50.5 -> 34.0 mm, vias 3 -> 0
- net CARD-SCLK: track 70.8 -> 55.3 mm, vias 3 -> 0
- net /LED1: track 61.4 -> 75.6 mm
- net /ADC-VOUT: track 33.4 -> 47.2 mm
- net CARD-MOSI: track 72.2 -> 59.2 mm
- net /UART-RX: track 39.6 -> 26.8 mm
- net /UART-TX: track 41.2 -> 29.6 mm
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- added copper zone on F.Cu, net GND
- added copper zone on F.Cu, net Net-(C10-Pad1)
- removed copper zone on B.Cu, net GNDA
- removed copper zone on B.Cu, net GNDPWR
- removed copper zone on F.Cu, net GNDPWR
- removed copper zone on F.Cu, net Net-(C10-Pad2)
Other:
- board text added: "DCPSU Card A v0.4-WIP"
- board text removed: "DCPSU Card A v0.3"
- board text removed: "SCL"
- board text removed: "SDA"

Commit message: Update Card A (v0.4-WIP)
Parts:
- added C12: 10u, Capacitor_SMD:C_1206_3216Metric_Pad1.42x1.75mm_HandSolder, F.Cu at (104.0, 106.0)
Routing:
- net GND: vias 50 -> 45
Other:
- outline, holes or cut-outs redrawn
