File: dcpsu-card-a.sch (KiCad schematic (older format))
At the start: 49 parts, among them J1 PCIe_x1, J2 Conn_01x06, J3 AVR-ISP-6, J4 Conn_01x02, U1 ATtiny87-MU, U2 AOZ2151PQI-10, U3 MCP4017T-104E_LT, U4 INA219AIDCNR

Commit message: Card A Rev 0.3
Parts:
- removed U3: MCP4017T-104E_LT, digikey-footprints:SOT-363, symbol dk_Data-Acquisition-Digital-Potentiometers:MCP4017T-103E_LT
- added C16: 0.1u, Capacitor_SMD:C_0603_1608Metric_Pad1.05x0.95mm_HandSolder, symbol Device:C
- added R23: 100, Resistor_SMD:R_0603_1608Metric_Pad1.05x0.95mm_HandSolder, symbol Device:R
- added U3: MCP4706A0T-E_CH, digikey-footprints:SOT-23-6, symbol dcpsu-custom-symbols:MCP4706A0T-E_CH
- C2: value 1u -> 10u; Digi-Key_PN 399-7847-1-ND -> 478-10766-1-ND
- C4, C5: Digi-Key_PN 399-1099-1-ND -> 1276-1000-1-ND
- J1: footprint Connector_PCBEdge:BUS_PCIexpress -> custom-footprints:BUS_PCIe_custom
- R10, R8: value 2k -> 0; Digi-Key_PN RMCF0603FT2K00CT-ND -> (none)
- R20: value 2k -> 3k; Digi-Key_PN RMCF0603FT2K00CT-ND -> (none)
- R6: value 2k -> 10k; Digi-Key_PN RMCF0603FT2K00CT-ND -> (none)
- R9: value 2k -> 47k; Digi-Key_PN RMCF0603FT2K00CT-ND -> (none)
- RN2: footprint Resistor_SMD:R_Array_Convex_4x1206 -> Resistor_SMD:R_Array_Convex_4x0612
Connections:
- net labels added: GNDPWR
- wire segments 274 -> 267
- no-connect marks 5 -> 6
Other:
- moved on the sheet: C2, C9, J1A, J1B, R1, R10, R19, R2, R3, R4, R5, R7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

Commit message: Update with notes and pending changes
Parts:
- R10: value 0 -> 3k
- R9: value 47k -> 43k
Other:
- note added: "LEDs too bright"
- note added: "R16 should be 1K!"
Changed lines of the file:
@@
 P 7150 2300
 F 0 "R9" H 7220 2346 50  0000 L CNN
-F 1 "47k" H 7220 2255 50  0000 L CNN
+F 1 "43k" H 7220 2255 50  0000 L CNN
 F 2 "Resistor_SMD:R_0603_1608Metric_Pad1.05x0.95mm_HandSolder" V 7080 2300 50  0001 C CNN
 F 3 "~" H 7150 2300 50  0001 C CNN
@@
 P 6800 2300
 F 0 "R10" H 6870 2346 50  0000 L CNN
-F 1 "0" H 6870 2255 50  0000 L CNN
+F 1 "3k" H 6870 2255 50  0000 L CNN
 F 2 "Resistor_SMD:R_0603_1608Metric_Pad1.05x0.95mm_HandSolder" V 6730 2300 50  0001 C CNN
 F 3 "~" H 6800 2300 50  0001 C CNN
@@
 Wire Wire Line
 	1000 3050 1000 3100
+Text Notes 8000 4900 0    50   ~ 0
+R16 should be 1K!
+Text Notes 5300 4700 0    50   ~ 0
+LEDs too bright
 $EndSCHEMATC

Commit message: Card A v0.4-WIP
Parts:
- removed C11, C12: 22u, Capacitor_SMD:C_1206_3216Metric_Pad1.42x1.75mm_HandSolder, symbol Device:C
- removed RN2: 220, Resistor_SMD:R_Array_Convex_4x0612, symbol Device:R_Pack04
- added C11: 100u, Capacitor_SMD:CP_Elec_6.3x7.7, symbol Device:CP
- added R24, R25: 2k, Resistor_SMD:R_0603_1608Metric_Pad1.05x0.95mm_HandSolder, symbol Device:R
- C10, C8: value 22u -> 10u; Digi-Key_PN 1276-3047-1-ND -> 1276-6736-1-ND
- R16: value 18k 0.1% -> 1k 0.1%; Digi-Key_PN P20113CT-ND -> P19972CT-ND
Connections:
- net GNDA is gone; now on net GND: C2.1, C4.2, J1.B11, R8.2, U2.3 (AGND)
- net GND: now also C10.2, C13.2, C6.2, C7.2, C8.2, D1.2 (A), J1.A1, J1.B1, J1.B10, J1.B2, J1.B3, J1.B4, J1.B5, J1.B6, J1.B7, J1.B8, J1.B9, J4.2 (Pin_2), R16.1, U2.10 (PGND), U2.11 (PGND), U2.12 (PGND), C11.2, R24.2, R25.2; no longer D2.2 (B_K)
- net LED2: now also D2.1 (B_A)
- net at R6.1, R7.1, U2.2 (FB): now also R10.1; no longer R10.2
- net at L1.2, R11.1, R12.1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: now also C10.1, C8.1, R9.2, C11.1; no longer C10.2, C8.2, R9.1
- net at D2.6 (G_K): now also R24.1
- removed net GNDPWR: C10.1, C13.2, C6.2, C7.2, C8.1, D1.2 (A), J1.A1, J1.B1, J1.B10, J1.B2, J1.B3, J1.B4, J1.B5, J1.B6, J1.B7, J1.B8, J1.B9, J4.2 (Pin_2), R16.1, U2.10 (PGND), U2.11 (PGND), U2.12 (PGND)
- new net: R10.2, R9.1
- new net: D2.2 (B_K), R25.1
- no-connect marks 6 -> 4
Other:
- note added: "Card edge connector"
- note added: "Debug connectors"
- note added: "Indicator LEDs"
- note added: "µC"
- note removed: "LEDs too bright"
- note removed: "R16 should be 1K!"
- moved on the sheet: C1, C10, C13, C3, C8, D1, D2A, D2B, D2C, J1A, J1B, J2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

Commit message: Update Card A (v0.4-WIP)
Parts:
- added C12: 10u, Capacitor_SMD:C_1206_3216Metric_Pad1.42x1.75mm_HandSolder, symbol Device:C
- J4: footprint Connector_Molex:Molex_Sabre_43160-1102_1x02_P7.49mm_Horizontal -> Connector_Molex:Molex_Nano-Fit_105313-xx02_1x02_P2.50mm_Horizontal
Connections:
- net +24V: now also C12.1
- net GND: now also C12.2
Changed lines of the file:
@@
 Comment2 "License: CC BY-SA"
 Comment3 "https://www.eevblog.com/projects/usupply/"
-Comment4 "Based on EEVblog's µSupply project"
+Comment4 "Inspired by EEVblog's µSupply project"
 $EndDescr
 $Comp
@@
 Wire Wire Line
 	5150 5950 5050 5950
-$Bitmap
-Pos 11050 7050
-Scale 1.000000
-Data
-89 50 4E 47 0D 0A 1A 0A 00 00 00 0D 49 48 44 52 00 00 00 58 00 00 00 1F 08 03 00 00 00 54 16 FA
-D2 00 00 00 03 73 42 49 54 08 08 08 DB E1 4F E0 00 00 01 BF 50 4C 54 45 FF FF FF 00 00 00 FF FF
-FF B5 BA B4 B7 BC B6 B9 BE B8 BC C1 BB BE C3 BE C1 C5 C0 C3 C8 C3 C6 CA C5 C8 CC C7 C9 CD C9 CB
-CE CA CC CF CB CC D0 CC CB CF CA CA CD C9 C4 C8 C3 BF C3 BE B9 BE B9 B3 B8 B2 B1 B7 B0 B0 B5 AF
-AE B4 AD AD B3 AC AC B2 AB AB B1 AA BA BF B9 BD C2 BC C0 C4 BF C3 C7 C2 C9 CD C8 CE D1 CD D0 D3
-CF D1 D4 D0 D2 D5 D2 D3 D6 D2 D1 D4 D1 CB CF CB C0 C5 BF AF B5 AE C0 C5 C0 C7 CB C7 84 85 84 43
-44 43 0D 0E 0D 84 86 84 CE D2 CE C4 C9 C4 BD C2 BD B2 B8 B1 B0 B6 AF AE B3 AD 79 7C 79 29 29 29
-CC D0 CB 91 93 91 1B 1B 1B 91 94 91 C5 C9 C4 B4 B9 B3 B2 B7 B1 93 98 93 28 29 28 40 40 40 70 70
-70 50 51 50 10 10 10 60 60 60 80 80 80 BF BF BF C4 C7 C3 CD D1 CC B6 BB B5 9F A3 9E 0E 0E 0E 50
-50 50 DF DF DF FF FF FF EF EF EF 9F 9F 9F BB C0 BA B8 BD B7 E3 E3 E3 C8 C7 C7 30 30 30 B1 B6 B0
-AF B4 AE D6 D5 D5 A3 A1 A1 23 1F 20 BA B9 B9 C8 CC C8 BF C4 BE B4 BA B3 3F 37 39 63 5F 61 76 73
-74 91 8F 8F CF CF CF BC C1 BC F1 F1 F1 9F 96 9A 8E 87 8B 9E 9D 9D 31 2D 2E CD D1 CD BE C2 BD 24
-24 24 28 28 28 E8 E7 E7 CF D3 CF 8F 8F 8F B5 B5 B5 2D 2D 2D E0 DF E0 AF AF AF BB C0 BB C9 C8 C8
-AC AB AB D2 D5 D1 20 20 20 84 81 82 2A 27 27 98 96 97 C6 CA C6 6E 6C 6C CB CA CB BA BF BA C2 C7
-C2 C5 C9 C5 9E A0 9D 7C 7F 7C 5D 5E 5D 82 85 82 70 72 6F D0 D4 D0 35 36 35 7D 7F 7C CD D0 CC 96
-99 96 32 33 31 AF B2 AF B0 B3 AF 3E 3F 3E 89 8C 89 BC C0 BC FF FF FF AA C0 F9 42 00 00 00 95 74
-52 4E 53 0E FF 00 FF FF FF FF FF FF FF FF FF FF FF FF FF FF FF FF FF FF FF FF FF FF FF FF FF FF
-FF FF FF FF FF FF FF FF FF FF FF FF FF FF FF FF FF FF FF FF FF FF FF FF FF FF FF FF FF FF FF FF
-FF FF FF FF FF FF FF FF FF FF FF FF FF FF FF FF FF FF FF FF FF FF FF FF FF FF FF FF FF FF FF FF
-FF FF FF FF FF FF FF FF FF FF FF FF FF FF FF FF FF FF FF FF FF FF FF FF FF FF FF FF FF FF FF FF
-FF FF FF FF FF FF FF FF FF FF FF FF FF FF FF FF FF FF FF FF FF FF FF 0A 7C 1A 13 92 00 00 03 80
-49 44 41 54 48 89 B5 96 89 5F 12 41 14 C7 79 09 84 BB 2E 10 9A 25 8A C0 AE 94 94 D0 2D 87 A5 2C
-72 74 C1 40 25 A5 6B DA 69 87 DD 65 29 76 A7 DD 97 D5 1F DC 9B 59 8E 65 81 3E 89 F5 3E F0 19 3E
-6F 76 BE BC F9 CD 7B 6F D6 60 80 FF 62 9B 90 DB 66 34 99 37 5B DA 39 BE 43 B0 DA 6C 56 FB 16 9E
-73 58 3A CD 5D C6 B6 AD DD DB B6 F7 F4 38 7B D7 6F 00 06 E4 F6 B9 FA DD 9C C7 EE 15 A5 01 9F 6F
-60 87 E8 DD E9 E1 DC 83 AE 3E 4A F6 6F EF 71 B6 44 36 00 72 77 39 76 0B 5E 69 28 10 A4 9B 08 06
-F6 48 7B ED FC 3E CB 7E 24 1F 38 E8 3F 54 0E 79 38 44 A7 43 C3 7A 46 43 3F 82 4D C8 E5 C3 62 24
-5A 15 28 3A 22 DA 3C 87 2D AE 2E E3 91 D1 83 A5 90 C7 62 00 72 3C 2E 03 C4 C6 B4 84 26 7E 04 9B
-FB 1D BC 4D 1A 47 5E 22 99 4A A7 53 C9 04 FE 1C 3F 7A CC B3 6F D0 6C 3A 8E 62 B0 90 4F 9C 84 4C
-96 A0 65 33 70 52 43 68 E6 47 F0 66 F7 EE 30 E5 26 52 39 A2 5A 1E D1 B1 A3 36 DE DD 79 EA 74 1B
-0B B9 B7 37 06 49 9C 01 A0 D3 10 AB 02 98 FF CC C4 C4 19 9D 1F C1 16 4E 10 91 5B C8 92 8A E5 0A
-18 B3 68 E7 2C 2E 0C F9 EC 39 D4 62 18 32 93 65 30 C9 40 45 4F E6 9F 52 D0 A6 6B FC 14 DC 7E DE
-1B 41 6E 8E 90 5A F2 C8 5E 8F 63 E6 94 71 76 D4 7F C8 E9 0C 81 E6 7F B3 10 2A AF A7 FE 09 E5 C2
-C5 4B 8A 72 59 EB A7 60 CE 2E 45 21 71 85 D4 58 2E 01 51 69 27 67 B9 6A C2 C4 40 2D 40 A6 DE 24
-30 41 88 0C 95 F5 32 99 BB A6 5C 27 E4 86 72 53 EB A7 60 7E 7E 08 20 45 74 96 07 D8 E3 E5 DD B7
-FA 50 0B 0A 8E 13 A6 84 AA 45 BC 0A 8E 93 B9 DB CA 1D 94 59 51 EE 6A FC 14 DC 71 2F 00 09 14 22
-9D 91 E5 94 3A DC C7 C5 09 08 88 5B A8 16 47 BA CF FD 11 4C 1E 3C 4C 33 F0 23 1D 58 90 82 74 83
-69 96 C1 F2 02 1B 92 74 DB C1 1D F6 C3 83 8F 4F CF 76 FB FF 28 05 99 9E 7A 42 C8 A2 A2 E8 A5 B0
-2E 01 60 88 05 28 66 D3 C5 7C 01 D3 63 A1 98 67 5A 0C 58 39 8B 19 13 0E C1 A5 C3 53 03 D6 1D DE
-0D 45 59 5E 7E AA 3C D3 1F 5E D8 07 90 A6 6B 52 EA D2 92 DC B8 03 9F ED 79 19 8C 69 55 05 D7 A6
-1B 21 CB 34 DD 5E CC E9 D3 ED AF C0 DA 02 89 D7 15 C8 CB C5 C5 49 9D BF 46 8A DC 95 62 0A A5 A0
-83 5E 8A 56 4A BA 74 78 A5 53 AB 1C 5E 1C 82 92 50 39 3C 24 60 B3 29 24 E3 05 7D 13 6A E2 67 E9
-36 0E 09 52 49 B7 05 99 0D A4 88 E9 D6 E1 98 79 A5 A6 1B D3 73 9D 6D 93 9F 8F 30 2D 1A 15 C8 EB
-5B 5D C7 B7 AA 5D 68 9D 86 E0 37 AC A4 B3 B5 5C 7D 49 B7 02 C6 26 B4 D2 A8 09 45 BC 9E F6 4E 2C
-3C D6 84 5A 01 C3 AA 20 BE 45 B2 A6 0D 65 59 DB 14 DE 6D E4 9A A6 B7 FF 7B EB 07 6D A3 CF A5 B0
-D1 7F 94 C2 AB 1B E1 32 30 7C B2 7D C0 98 6B AE 26 E9 F3 17 DD 93 6A 7D 80 FA AD 9F D0 7B D5 F7
-95 4F 56 71 45 7B 99 46 C4 B0 9E 0B A4 F4 A9 E3 56 27 EB C1 F0 1E AF FF 48 F9 FA 1F 91 BC 42 BD
-0E E5 B6 D9 60 42 6D 21 0D C1 F0 F5 9B 7D FE 9E B4 E4 F3 2D 49 F8 C2 F2 7D AD 6E 39 34 11 42 9D
-6A 1A 31 DA DA 8F 9F 82 35 1C B6 0A 3F 7F 34 C0 36 8F B8 AC 7D 53 F0 3F 36 C3 AF FF C3 DD F4 1B
-58 55 66 0F 67 B9 51 C4 00 00 00 00 49 45 4E 44 AE 42 60 82
-EndData
-$EndBitmap
 $Bitmap
 Pos 6600 7400
@@
 F 0 "J4" H 10280 2792 50  0000 L CNN
 F 1 "Conn_01x02" H 10280 2701 50  0000 L CNN
-F 2 "Connector_Molex:Molex_Sabre_43160-1102_1x02_P7.49mm_Horizontal" H 10200 2800 50  0001 C CNN
+F 2 "Connector_Molex:Molex_Nano-Fit_105313-xx02_1x02_P2.50mm_Horizontal" H 10200 2800 50  0001 C CNN
 F 3 "~" H 10200 2800 50  0001 C CNN
 F 4 "WM18483-ND" H 10200 2800 50  0001 C CNN "Digi-Key_PN"
@@
 L power:GNDPWR #PWR0102
 U 1 1 5FD9C4DB
-P 6600 1500
-F 0 "#PWR0102" H 6600 1300 50  0001 C CNN
-F 1 "GNDPWR" H 6604 1346 50  0000 C CNN
-F 2 "" H 6600 1450 50  0001 C CNN
-F 3 "" H 6600 1450 50  0001 C CNN
-	1    6600 1500
+P 6950 1500
+F 0 "#PWR0102" H 6950 1300 50  0001 C CNN
+F 1 "GNDPWR" H 6954 1346 50  0000 C CNN
+F 2 "" H 6950 1450 50  0001 C CNN
+F 3 "" H 6950 1450 50  0001 C CNN
+	1    6950 1500
 	1    0    0    -1
 $EndComp
@@
 Wire Wire Line
 	7400 2450 7750 2450
-Wire Wire Line
-	6600 1450 6600 1500
 Connection ~ 6600 1450
 Wire Wire Line
@@
 Wire Wire Line
 	6900 2050 6900 3250
+$Comp
+L Device:C C12
+U 1 1 60206501
+P 6950 1250
+F 0 "C12" H 7065 1296 50  0000 L CNN
+F 1 "10u" H 7065 1205 50  0000 L CNN
+F 2 "Capacitor_SMD:C_1206_3216Metric_Pad1.42x1.75mm_HandSolder" H 6988 1100 50  0001 C CNN
+F 3 "" H 6950 1250 50  0001 C CNN
+F 4 "1276-6736-1-ND" H 6950 1250 50  0001 C CNN "Digi-Key_PN"
+	1    6950 1250
+	1    0    0    -1
+$EndComp
+Wire Wire Line
+	6600 1050 6950 1050
+Wire Wire Line
+	6950 1050 6950 1100
+Connection ~ 6600 1050
+Wire Wire Line
+	6600 1450 6950 1450
+Wire Wire Line
+	6950 1450 6950 1500
+Wire Wire Line
+	6950 1400 6950 1450
+Connection ~ 6950 1450
 $EndSCHEMATC
