File: backplane-testboard/backplane-testboard.sch (KiCad schematic (older format))
At the start: 38 parts, among them J1 Conn_01x02, J10 Conn_01x01_Female, J11 10018784-10201TLF, J12 Conn_01x01_Female, J13 Conn_01x08_Female, J2 AVR-ISP-6, J3 Conn_01x02, J4 Conn_01x08_Female, J5 Conn_01x01_Female, J6 10018784-10201TLF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

Commit message: Update with 1U chassis backplane and Card A v0.4
Parts:
- J11, J6: symbol PCIe-connector-symbol:10018784-10201TLF -> 10018784-10201TLF:10018784-10201TLF
Changed lines of the file:
@@
 $EndDescr
 $Comp
-L PCIe-connector-symbol:10018784-10201TLF J6
+L 10018784-10201TLF:10018784-10201TLF J6
 U 1 1 5F440570
 P 6400 4500
@@
 	6900 6100 7050 6100
 $Comp
-L PCIe-connector-symbol:10018784-10201TLF J11
+L 10018784-10201TLF:10018784-10201TLF J11
 U 1 1 5F55ED3C
 P 9400 4500
