File: dcpsu-card-a-ti/dcpsu-card-a.sch (KiCad schematic (older format))
At the start: 52 parts, among them J1 PCIe_x1, J2 Conn_01x06, J3 AVR-ISP-6, J4 Conn_01x02, U1 ATtiny87-MU, U2 AOZ2151PQI-10, U3 MCP4706A0T-E_CH, U4 INA219AIDCNR

Commit message: Update with 1U chassis backplane and Card A v0.4
Parts:
- removed R7: 2k, Resistor_SMD:R_0603_1608Metric_Pad1.05x0.95mm_HandSolder, symbol Device:R
- removed R8: 0, Resistor_SMD:R_0603_1608Metric_Pad1.05x0.95mm_HandSolder, symbol Device:R
- removed U2: AOZ2151PQI-10, custom-footprints:QFN-20-2EP_3x3mm_AOZ2151PQI-10, symbol dcpsu-custom-symbols:AOZ2151PQI-10
- added D3, D4: D_Schottky, custom-footprints:TO-277B-MBR860S, symbol Device:D_Schottky
- added D5: D_TVS, Diode_SMD:D_0201_0603Metric, symbol Device:D_TVS
- added POT1: TC33X-1-502E, digikey-footprints:Trimpot_3.8mmx3.6mm_TC33X-2-103E, symbol dk_Trimmer-Potentiometers:TC33X-2-103E
- added R29: 33k, Resistor_SMD:R_0603_1608Metric_Pad1.05x0.95mm_HandSolder, symbol Device:R
- added U2: LMR33640, Package_SO:TI_SO-PowerPAD-8, symbol dcpsu-custom-symbols:LMR33640
- C11: Digi-Key_PN (none) -> 732-8511-1-ND
- C13, C14, C15, C16, C3, C9: value 0.1u -> 0.1u 16V
- C2: value 10u -> 1u; Digi-Key_PN 478-10766-1-ND -> 399-7847-1-ND
- C4: value 0.1u -> C; Digi-Key_PN 1276-1000-1-ND -> (none)
- C5: value 0.1u -> 0.1u 50V
- C6: value 10u -> 0.1u 50V; footprint Capacitor_SMD:C_1206_3216Metric_Pad1.42x1.75mm_HandSolder -> Capacitor_SMD:C_0603_1608Metric_Pad1.05x0.95mm_HandSolder; Digi-Key_PN 1276-6736-1-ND -> 1276-1000-1-ND
- J4: Digi-Key_PN WM18483-ND -> WM14972-ND
- L1: value 10uH -> 15uH; footprint custom-footprints:L_Pad4.05x4.4mm_LMLP1011 -> dcpsu-custom-footprints:L_9.5x9.0_H4.0; Digi-Key_PN 478-LMLP1011M100DTASCT-ND -> P19773CT-ND
- R10: value 3k -> 10k; Digi-Key_PN (none) -> RMCF0603JT10K0CT-ND
- R20: value 3k -> 2k; Digi-Key_PN (none) -> RMCF0603FT2K00CT-ND
- R23: Digi-Key_PN (none) -> RMCF0603JT100RCT-ND
- R6: Digi-Key_PN (none) -> RMCF0603JT10K0CT-ND
- R9: value 43k -> 33k; Digi-Key_PN (none) -> RMCF0603JT33K0CT-ND
Connections:
- net labels added: PWR-GOOD
- net labels removed: PWR-PWM
- wire segments 271 -> 287
- no-connect marks 4 -> 5
Other:
- moved on the sheet: C12, C16, C5, C6, C7, C9, L1, R10, R2, R20, R3, R4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
